File: Mushroom_hw/LedPcb.sch (KiCad schematic (older format))
At the start: 6 parts, among them Q1 LED_RGB, Q2 LED_RGB_WS2812B

Commit message: + New LedPcb (WS2812 only)
Parts:
- removed Q1: LED_RGB, ~, symbol LED_RGB
- removed XL1, XL2: CONN_3, ~, symbol CONN_3
- added HOLE1: HOLE_METALLED, PCB:Hole1d8_out3d2mm, symbol HOLE_METALLED
- added XL1, XL2, XL4, XL5, XL6: CONN_1, PCB:Oval3x1.5, symbol CONN_1
- C1: footprint CAP_0603 -> Capacitors:CAP_0603
- Q1: renamed from Q2; footprint ~ -> LEDs:LED_WS2812B
- XL3: footprint ~ -> PCB:Oval3x1.5
Connections:
- net labels added: DIN, DOUT, GND, VDD
- wire segments 31 -> 17
Changed lines of the file:
@@
 LIBS:Connectors_kl
 LIBS:Tittar_kl
+LIBS:pcb_details
 LIBS:LedPcb-cache
-EELAYER 27 0
+EELAYER 26 0
 EELAYER END
 $Descr A4 11693 8268
@@
 $EndDescr
 $Comp
-L LED_RGB Q1
-U 1 1 532DF73F
-P 4000 2400
-F 0 "Q1" H 3800 2750 60  0000 C CNN
-F 1 "LED_RGB" H 4150 2750 60  0000 C CNN
-F 2 "~" H 4000 2400 60  0000 C CNN
-F 3 "~" H 4000 2400 60  0000 C CNN
-	1    4000 2400
-	1    0    0    -1
-$EndComp
-$Comp
-L LED_RGB_WS2812B Q2
+L LED_RGB_WS2812B Q1
 U 1 1 532DF74E
 P 4000 3450
-F 0 "Q2" H 3800 3800 60  0000 C CNN
+F 0 "Q1" H 3800 3800 60  0000 C CNN
 F 1 "LED_RGB_WS2812B" H 4000 3700 60  0000 C CNN
-F 2 "~" H 3950 3450 60  0000 C CNN
+F 2 "LEDs:LED_WS2812B" H 3950 3450 60  0001 C CNN
 F 3 "~" H 3950 3450 60  0000 C CNN
 	1    4000 3450
-	1    0    0    -1
-$EndComp
-$Comp
-L CONN_1 XL3
-U 1 1 532ED359
-P 5250 3550
-F 0 "XL3" V 5200 3560 40  0000 C CNN
-F 1 "CONN_1" V 5260 3570 40  0000 C CNN
-F 2 "~" H 5250 3550 60  0000 C CNN
-F 3 "~" H 5250 3550 60  0000 C CNN
-	1    5250 3550
 	1    0    0    -1
 $EndComp
@@
 F 0 "C1" V 3900 3700 50  0000 L CNN
 F 1 "0.1u" V 3900 3950 50  0000 L CNN
-F 2 "CAP_0603" V 4100 3700 28  0000 C BNN
+F 2 "Capacitors:CAP_0603" V 4100 3700 28  0001 C BNN
 F 3 "~" H 4000 3850 60  0000 C CNN
 	1    4000 3850
 	0    -1   -1   0
-$EndComp
-$Comp
-L CONN_3 XL1
-U 1 1 532ED892
-P 2600 2400
-F 0 "XL1" V 2550 2400 40  0000 C CNN
-F 1 "CONN_3" V 2650 2400 40  0000 C CNN
-F 2 "~" H 2600 2400 60  0000 C CNN
-F 3 "~" H 2600 2400 60  0000 C CNN
-	1    2600 2400
-	1    0    0    -1
-$EndComp
-$Comp
-L CONN_3 XL2
-U 1 1 532ED8A1
-P 5250 2400
-F 0 "XL2" V 5200 2400 40  0000 C CNN
-F 1 "CONN_3" V 5300 2400 40  0000 C CNN
-F 2 "~" H 5250 2400 60  0000 C CNN
-F 3 "~" H 5250 2400 60  0000 C CNN
-	1    5250 2400
-	-1   0    0    -1
 $EndComp
 Wire Wire Line
@@
 Wire Wire Line
 	2950 3550 3550 3550
+Connection ~ 3500 3550
+$Comp
+L CONN_1 XL4
+U 1 1 5961F8CC
+P 5250 3150
+F 0 "XL4" V 5200 3160 40  0000 C CNN
+F 1 "CONN_1" V 5260 3170 40  0000 C CNN
+F 2 "PCB:Oval3x1.5" H 5250 3150 60  0001 C CNN
+F 3 "~" H 5250 3150 60  0000 C CNN
+	1    5250 3150
+	1    0    0    -1
+$EndComp
+$Comp
+L CONN_1 XL5
+U 1 1 5961FACC
+P 5250 3900
+F 0 "XL5" V 5200 3910 40  0000 C CNN
+F 1 "CONN_1" V 5260 3920 40  0000 C CNN
+F 2 "PCB:Oval3x1.5" H 5250 3900 60  0001 C CNN
+F 3 "~" H 5250 3900 60  0000 C CNN
+	1    5250 3900
+	1    0    0    -1
+$EndComp
+$Comp
+L CONN_1 XL1
+U 1 1 5961FB0F
+P 2750 3200
+F 0 "XL1" V 2700 3210 40  0000 C CNN
+F 1 "CONN_1" V 2760 3220 40  0000 C CNN
+F 2 "PCB:Oval3x1.5" H 2750 3200 60  0001 C CNN
+F 3 "~" H 2750 3200 60  0000 C CNN
+	1    2750 3200
+	-1   0    0    -1
+$EndComp
+$Comp
+L CONN_1 XL2
+U 1 1 5961FB79
+P 2750 3550
+F 0 "XL2" V 2700 3560 40  0000 C CNN
+F 1 "CONN_1" V 2760 3570 40  0000 C CNN
+F 2 "PCB:Oval3x1.5" H 2750 3550 60  0001 C CNN
+F 3 "~" H 2750 3550 60  0000 C CNN
+	1    2750 3550
+	-1   0    0    -1
+$EndComp
 Wire Wire Line
-	2800 2500 2800 2550
+	3550 3350 3300 3350
 Wire Wire Line
-	2800 2550 3600 2550
+	3300 3350 3300 3200
 Wire Wire Line
-	5050 2500 5050 2550
+	3300 3200 2950 3200
 Wire Wire Line
-	5050 2550 4400 2550
-Connection ~ 3500 3550
+	5050 3150 4800 3150
 Wire Wire Line
-	4450 3350 4450 2950
+	4800 3150 4800 3350
 Wire Wire Line
-	4450 2950 3400 2950
+	4800 3350 4450 3350
 Wire Wire Line
-	3550 3350 3550 2850
+	5050 3900 4800 3900
 Wire Wire Line
-	3550 2850 4650 2850
+	4800 3550 4800 4250
+Connection ~ 4800 3550
+Text Label 3350 3350 0    60   ~ 0
+DIN
+Text Label 4500 3350 0    60   ~ 0
+DOUT
+Text Label 3250 3550 0    60   ~ 0
+VDD
+Text Label 4550 3550 0    60   ~ 0
+GND
+$Comp
+L CONN_1 XL3
+U 1 1 59620078
+P 2750 3900
+F 0 "XL3" V 2700 3910 40  0000 C CNN
+F 1 "CONN_1" V 2760 3920 40  0000 C CNN
+F 2 "PCB:Oval3x1.5" H 2750 3900 60  0001 C CNN
+F 3 "~" H 2750 3900 60  0000 C CNN
+	1    2750 3900
+	-1   0    0    -1
+$EndComp
 Wire Wire Line
-	3150 2250 3150 2400
+	2950 3900 3050 3900
 Wire Wire Line
-	3150 2400 2800 2400
+	3050 3900 3050 3550
+Connection ~ 3050 3550
+$Comp
+L CONN_1 XL6
+U 1 1 5962014D
+P 5250 4250
+F 0 "XL6" V 5200 4260 40  0000 C CNN
+F 1 "CONN_1" V 5260 4270 40  0000 C CNN
+F 2 "PCB:Oval3x1.5" H 5250 4250 60  0001 C CNN
+F 3 "~" H 5250 4250 60  0000 C CNN
+	1    5250 4250
+	1    0    0    -1
+$EndComp
 Wire Wire Line
-	2800 2300 3050 2300
-Wire Wire Line
-	3050 2300 3050 2350
-Wire Wire Line
-	3050 2350 3250 2350
-Wire Wire Line
-	3250 2350 3250 2400
-Wire Wire Line
-	3250 2400 3600 2400
-Wire Wire Line
-	3150 2250 3600 2250
-Wire Wire Line
-	3400 2950 3400 2400
-Connection ~ 3400 2400
-Wire Wire Line
-	2950 3550 2950 2550
-Connection ~ 2950 2550
-Wire Wire Line
-	4650 2850 4650 2550
-Connection ~ 4650 2550
-Wire Wire Line
-	4400 2250 4900 2250
-Wire Wire Line
-	4900 2250 4900 2400
-Wire Wire Line
-	4900 2400 5050 2400
-Wire Wire Line
-	5050 2300 4800 2300
-Wire Wire Line
-	4400 2400 4800 2400
-Wire Wire Line
-	4800 2400 4800 2300
+	4800 4250 5050 4250
+Connection ~ 4800 3900
+$Comp
+L HOLE_METALLED HOLE1
+U 1 1 5962038C
+P 5350 3550
+F 0 "HOLE1" H 5100 3600 60  0000 C CNN
+F 1 "HOLE_METALLED" H 4900 3500 60  0000 C CNN
+F 2 "PCB:Hole1d8_out3d2mm" H 4750 3400 60  0001 C CNN
+F 3 "" H 4850 3500 60  0001 C CNN
+F 4 "0" H 4950 3600 60  0001 C CNN "Price"
+F 5 "0" H 5050 3700 60  0001 C CNN "SolderPoints"
+	1    5350 3550
+	-1   0    0    -1
+$EndComp
 $EndSCHEMATC
