File: Mushroom_hw/mushroom.sch (KiCad schematic (older format))
At the start: 129 parts, among them Q1 LED_RGB_WS2812B, Q2 LED_RGB, Q3 LED_RGB_WS2812B, Q4 LED_RGB, Q5 LED_RGB, Q6 LED_RGB_WS2812B, SW1 SWITCH_H

Commit message: HW v1 for archive purposes
Parts:
- ANT1: symbol ANT_PCB_NOCNTR -> ANT_PCB_NoCntr
- D1, D2, D3: symbol D_SHOTTKY -> D_Shottky
- DD1: symbol STM32L151CXTX -> STM32L151CxTx
- F1, F10, F11, F12, F13, F14, F15, F16, F17, F18, F19, F2, F20, F3, F4, F5, F6, F7, F8, F9: symbol FUSE0R -> Fuse0R
- HOLE1, HOLE2, HOLE3, HOLE4: symbol HOLE_METALLED -> HOLE_METALLED-RESCUE-mushroom
Changed lines of the file:
@@
 EESchema Schematic File Version 2
+LIBS:mushroom-rescue
 LIBS:Antennas_kl
 LIBS:Connectors_kl
@@
 LIBS:memory
 LIBS:mushroom-cache
-EELAYER 27 0
+EELAYER 25 0
 EELAYER END
 $Descr A2 23386 16535
@@
 $EndComp
 $Comp
-L STM32L151CXTX DD1
+L STM32L151CxTx DD1
 U 1 1 52A19E0D
 P 6000 2850
@@
 $EndComp
 $Comp
-L D_SHOTTKY D1
+L D_Shottky D1
 U 1 1 53288AAF
 P 4200 6300
@@
 $EndComp
 $Comp
-L D_SHOTTKY D2
+L D_Shottky D2
 U 1 1 532AFFD7
 P 9000 6300
@@
 $EndComp
 $Comp
-L D_SHOTTKY D3
+L D_Shottky D3
 U 1 1 532B006F
 P 13750 6300
@@
 $EndComp
 $Comp
-L FUSE0R F1
+L Fuse0R F1
 U 1 1 532EF061
 P 9750 12600
@@
 $EndComp
 $Comp
-L FUSE0R F2
+L Fuse0R F2
 U 1 1 532EF1BF
 P 10450 12600
@@
 $EndComp
 $Comp
-L FUSE0R F3
+L Fuse0R F3
 U 1 1 532EF1D3
 P 11150 12600
@@
 $EndComp
 $Comp
-L FUSE0R F7
+L Fuse0R F7
 U 1 1 532EF1E7
 P 12200 12600
@@
 $EndComp
 $Comp
-L FUSE0R F11
+L Fuse0R F11
 U 1 1 532EF1FB
 P 13250 12600
@@
 $EndComp
 $Comp
-L FUSE0R F4
+L Fuse0R F4
 U 1 1 532F0D37
 P 11500 13800
@@
 $EndComp
 $Comp
-L FUSE0R F5
+L Fuse0R F5
 U 1 1 532F0D3D
 P 11650 13800
@@
 $EndComp
 $Comp
-L FUSE0R F6
+L Fuse0R F6
 U 1 1 532F0D43
 P 11800 13800
@@
 $EndComp
 $Comp
-L FUSE0R F8
+L Fuse0R F8
 U 1 1 532F0D61
 P 12550 13800
@@
 $EndComp
 $Comp
-L FUSE0R F9
+L Fuse0R F9
 U 1 1 532F0D67
 P 12700 13800
@@
 $EndComp
 $Comp
-L FUSE0R F10
+L Fuse0R F10
 U 1 1 532F0D6D
 P 12850 13800
@@
 $EndComp
 $Comp
-L FUSE0R F13
+L Fuse0R F13
 U 1 1 532F40F9
 P 19350 11950
@@
 $EndComp
 $Comp
-L FUSE0R F12
+L Fuse0R F12
 U 1 1 532F4104
 P 19350 11750
@@
 $EndComp
 $Comp
-L FUSE0R F14
+L Fuse0R F14
 U 1 1 532F410A
 P 19350 12150
@@
 Connection ~ 20000 11200
 $Comp
-L FUSE0R F16
+L Fuse0R F16
 U 1 1 532F4C93
 P 20450 11950
@@
 $EndComp
 $Comp
-L FUSE0R F15
+L Fuse0R F15
 U 1 1 532F4C99
 P 20450 11750
@@
 $EndComp
 $Comp
-L FUSE0R F17
+L Fuse0R F17
 U 1 1 532F4C9F
 P 20450 12150
@@
 BLUE_N
 $Comp
-L FUSE0R F19
+L Fuse0R F19
 U 1 1 532F5A80
 P 20600 13850
@@
 $EndComp
 $Comp
-L FUSE0R F18
+L Fuse0R F18
 U 1 1 532F5A86
 P 20600 13650
@@
 $EndComp
 $Comp
-L FUSE0R F20
+L Fuse0R F20
 U 1 1 532F5A8C
 P 20600 14050
@@
 $EndComp
 $Comp
-L HOLE_METALLED HOLE3
+L HOLE_METALLED-RESCUE-mushroom HOLE3
 U 1 1 532F97A0
 P 4900 15000
@@
 $EndComp
 $Comp
-L HOLE_METALLED HOLE2
+L HOLE_METALLED-RESCUE-mushroom HOLE2
 U 1 1 532F97A6
 P 4900 14750
@@
 $EndComp
 $Comp
-L HOLE_METALLED HOLE1
+L HOLE_METALLED-RESCUE-mushroom HOLE1
 U 1 1 532F97AC
 P 4900 14500
@@
 Connection ~ 5300 14750
 $Comp
-L HOLE_METALLED HOLE4
+L HOLE_METALLED-RESCUE-mushroom HOLE4
 U 1 1 532F97B6
 P 4900 15250
@@
 Connection ~ 5300 15250
 $Comp
-L ANT_PCB_NOCNTR ANT1
+L ANT_PCB_NoCntr ANT1
 U 1 1 5332D14D
 P 14550 1800

Commit message: * HW v2 in progress
Parts:
- removed ANT1: ANT_PCB_NOCNTR, ~, symbol ANT_PCB_NoCntr
- removed B1, B2, B3: BAT, symbol BAT
- removed C25, C27: 220pF, symbol C
- removed C26: 0.1u, symbol C
- removed C28: 10u, symbol C
- removed D1, D2, D3: SS14, ~, symbol D_Shottky
- removed DA1, DA3, DA4: TPS61042, symbol TPS61042
- removed DD2: CC2500, symbol CC2500
- removed F10, F11, F12, F13, F14, F15, F16, F17, F18, F19, F2, F20, F3, F4, F5, F6, F7, F8, F9: FUSE0R, ~, symbol Fuse0R
- removed L3: 6.8uH, IND_1210, symbol L
- removed Q2, Q4, Q5: LED_RGB, ~, symbol LED_RGB
- removed R10, R9: 390k, RES_0603, symbol R
- removed R11, R16: 10k, RES_0603, symbol R
- removed R12, R17: 13R, RES_0603, symbol R
- removed R13, R18: 120k, RES_0603, symbol R
- removed R14: 56k, symbol R
- removed R15, R8: 100k, symbol R
- removed R19, R20, R21: 51R, RES_0603, symbol R
- removed SW1: SWITCH_H, ~, symbol SWITCH_H
- removed TP3: TESTPOINT, symbol TESTPOINT
- removed XL1, XL12, XL13, XL16, XL17, XL20, XL21, XL24, XL5, XL8, XL9: CONN_3, ~, symbol CONN_3
- removed XL2: ST_SWD, symbol ST_SWD
- removed XL3: CONN_4, symbol CONN_4
- removed XL4: CONN_4, ~, symbol CONN_4
- added ANT1: ANT_PCB_MONO, Radio:ANT_868_ARMLETG, symbol ANT_PCB_MONO
- added BLN1: BALUN868JOHANSON, Radio:BALUN_JOHANSON868, symbol BALUN868JOHANSON
- added DA1: MC74VHC1, SOT:SOT23-5, symbol MC74VHC1
- added DD2: CC1101, QFN_DFN:QFN20, symbol CC1101
- added HOLE5, HOLE6: HOLE_METALLED, PCB:Hole2d4_out4d5mm, symbol HOLE_METALLED-RESCUE-mushroom
- added Logo1: Logo, Pictures:Ostranna_12d7_10d1, symbol Logo
- added Q2: 2N7002, SOT:SOT23-3, symbol N_3PIN
- added Q4: IRLML9303, SOT:SOT23-3, symbol P_3PIN
- added RP3, RP4: REFPOINT, PCB:REF_POINT_1MM, symbol REFPOINT
- added SW1: SWITCH, Switches:SW_SS-1P2T, symbol SWITCH
- added SW2, SW3, SW4: BUTTON, BtnsSwitches:BTN_6x6_4x4, symbol BUTTON
- added XL1: CONN_6, Connectors:PLS-6, symbol CONN_6
- added XL2: CONN_1, Connectors:PLS-1Rnd, symbol CONN_1
- added XL3: CONN_2, Connectors:W02_Pitch_2d54, symbol CONN_2
- C1, C19: value 0.1u -> 10u; footprint (none) -> Capacitors:CAP_0603; PN (none) -> CL10A106MQ8NNNC; Price (none) -> 2.5; SolderPoints (none) -> 2; URL (none) -> https://www.terraelectronica.ru/catalog.php?ID=1155&search=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
- C10: value 1u -> 10n; footprint CAP_0603 -> Capacitors:CAP_0603
- C11: value 10u -> 10n; footprint (none) -> Capacitors:CAP_0603
- C12, C13, C14, C6, C8: footprint (none) -> Capacitors:CAP_0603
- C15: value 10u -> 1u; footprint (none) -> Capacitors:CAP_0603
- C16, C2: value 10u -> 220pF; footprint (none) -> Capacitors:CAP_0603
- C17, C18: value 10pF -> 18pF; footprint CAP_0603 -> Capacitors:CAP_0603; Price (none) -> 0.5; SolderPoints (none) -> 2
- C20: footprint (none) -> Capacitors:CAP_0603; Price (none) -> 0.5; SolderPoints (none) -> 2
- C21: footprint (none) -> Capacitors:CAP_0603; PN (none) -> CL10A106MQ8NNNC; Price (none) -> 2.5; SolderPoints (none) -> 2; URL (none) -> https://www.terraelectronica.ru/catalog.php?ID=1155&search=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
- C22: value 220pF -> 0.1u; footprint (none) -> Capacitors:CAP_0603
- C23, C24: value 0.1u -> *; footprint (none) -> Capacitors:CAP_0402; Price (none) -> 0.5; SolderPoints (none) -> 2
- C29, C30, C31, C5: footprint CAP_0603 -> Capacitors:CAP_0603
- C3: value 10u -> 0.1u; footprint CAP_0603 -> Capacitors:CAP_0603
- C4: value 0.1u -> 10n; footprint CAP_0603 -> Capacitors:CAP_0603
- C7: value 0.1u -> 3.3pF; footprint CAP_0603 -> Capacitors:CAP_0603
- C9: value 10n -> 0.1u; footprint CAP_0603 -> Capacitors:CAP_0603
- DA2: footprint ~ -> SOT:SC89-3
- DD1: value STM32L151CXTX -> STM32L151CxTx; footprint ~ -> LQFP_TQFP:LQFP48; PN (none) -> stm32L151c8t6; SolderPoints (none) -> 48; URL (none) -> http://
- F1: value FUSE0R -> Fuse0R; footprint ~ -> (none); Price (none) -> 0; SolderPoints (none) -> 1
- HOLE1, HOLE2, HOLE3, HOLE4: footprint (none) -> PCB:Hole2d4_out4d5mm
- L1: value 6.8uH -> BLM15AG102SN1; footprint IND_1210 -> Inductors:IND_0402
- L2: value 6.8uH -> *; footprint IND_1210 -> Inductors:IND_0402; Price (none) -> 4; SolderPoints (none) -> 2
- Q1, Q3, Q6: footprint ~ -> LEDs:LED_WS2812B
- R1: value 4K7 -> 100k; footprint RES_0402 -> Resistors:RES_0603; Price (none) -> 0.5; SolderPoints (none) -> 2
- R2: value 4K7 -> 100k; footprint RES_0402 -> Resistors:RES_0603
- R3: footprint (none) -> Resistors:RES_0603
- R4: value 150 -> 10k; footprint RES_0402 -> Resistors:RES_0603; Price (none) -> 0.5; SolderPoints (none) -> 2
- R5: value 10k -> 56k; footprint RES_0603 -> Resistors:RES_0603; Price (none) -> 0.5; SolderPoints (none) -> 2
- R6: value 13R -> 10k; footprint RES_0603 -> Resistors:RES_0603; Price (none) -> 0.5; SolderPoints (none) -> 2
- R7: value 120k -> 20k; footprint RES_0603 -> Resistors:RES_0603; Price (none) -> 0.5; SolderPoints (none) -> 2
- RP1, RP2: footprint (none) -> PCB:REF_POINT_1MM
- TP1, TP2: footprint (none) -> PCB:TESTPOINT_1MM; Price (none) -> 0; SolderPoints (none) -> 0
- XL10, XL11, XL14, XL15, XL18, XL19, XL22, XL23, XL6, XL7: footprint ~ -> (none)
- XTAL1: footprint 03225 -> Quartz:03225C4; Price (none) -> 15; SolderPoints (none) -> 4
Connections:
- net labels added: ADC_BATTERY, ANT1, ANT2, BTN1, BTN2, BTN3, NO_RADIO, PWR_EN, PwrUnst, RF1, RF2, VCC, WS_CTRL
- net labels removed: Ant, BLUE_N, BLUE_P, BLUE_PWM, BRIGHTNESS, CC_GDO2, GREEN_N, GREEN_P, GREEN_PWM, P_SCL, P_SDA, PeriphPwr, PeriphPwr1, RED_N, RED_P, RED_PWM
- wire segments 343 -> 199
- no-connect marks 18 -> 25
Other:
- note added: "Balun"
- note added: "Buttons"
- note added: "CC Power Filter"
- note added: "Extra transistor is required \nto eliminate fantom powering of MCU"
- note added: "Keep CS High\nwhen sleeping"
- note added: "MCU Power Filter"
- note added: "Matching circuit"
- note added: "Pins 15, 14, 11, 9, 4, 18"
- note added: "Pins 24, 36, 48, 1+9"
- note added: "Power switch"
- note added: "Programming & debug"
- note added: "Radio"
- note added: "Solder when radio not mounted\nto disable power-on check"
- note added: "WS2812 control"
- note removed: "Battery\nmeasurement"
- note removed: "Choose capacitor \nmax voltage carefully\n(30v recommended)"
- note removed: "For RGB"
- note removed: "For WS2812B"
- note removed: "Just\nPins"
- note removed: "Peripheral\nI2C Pull-Ups"
- note removed: "Pill"
- note removed: "Pill \nConnector"
- note removed: "Place resistors and fuses \nif single LED is required"
- note removed: "Programming"
- note removed: "R=252/Iled[mA]"
- note removed: "Solder fuses \nfor WS2812B"
- note removed: "UART"
- moved on the sheet: C12, C13, C29, C30, C31, C6, C8, DA2, Q1, Q3, Q6, RP1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

Commit message: + Component placement done
Parts:
- removed DA2: NCP583SQ, SOT:SC89-3, symbol NCP583SQ
- removed HOLE1, HOLE2, HOLE3, HOLE4, HOLE5, HOLE6: HOLE_METALLED, PCB:Hole2d4_out4d5mm, symbol HOLE_METALLED-RESCUE-mushroom
- added C23: 0.1u, Capacitors:CAP_0603, symbol C
- added DA1: NCP583SQ, SOT:SC82AB, symbol NCP583SQ
- added HOLE1, HOLE2, HOLE3, HOLE4, HOLE5, HOLE6: HOLE_METALLED, PCB:Hole2d4_out4d5mm, symbol HOLE_METALLED
- added Q3: ALS-PT19-315C, Resistors:RES_0603, symbol Phototransistor
- added R8: 10k, Resistors:RES_0603, symbol R
- F1: footprint (none) -> Resistors:RES_0603_FUSE
- R4: value 10k -> 100k
- SW1: footprint Switches:SW_SS-1P2T -> BtnsSwitches:SW_SS-1P2T
- XL10: renamed from XL18; footprint (none) -> Connectors:PLS-3
- XL11: renamed from XL19; footprint (none) -> Connectors:SIL1_ROUND_1MM8
- XL12: renamed from XL22; footprint (none) -> Connectors:PLS-3
- XL13: renamed from XL23; footprint (none) -> Connectors:SIL1_ROUND_1MM8
- XL4: renamed from XL6; footprint (none) -> Connectors:PLS-3
- XL5: renamed from XL7; footprint (none) -> Connectors:SIL1_ROUND_1MM8
- XL6: renamed from XL10; footprint (none) -> Connectors:PLS-3
- XL7: renamed from XL11; footprint (none) -> Connectors:SIL1_ROUND_1MM8
- XL8: renamed from XL14; footprint (none) -> Connectors:PLS-3
- XL9: renamed from XL15; footprint (none) -> Connectors:SIL1_ROUND_1MM8
- renumbered C8 to C10, C14 to C12, C15 to C13, C16 to C14, C12 to C15, C13 to C16, C19 to C18, C18 to C19, C21 to C20, C20 to C21, C23 to C24, C29 to C25, C24 to C26, C30 to C27, C31 to C28, C7 to C6, C6 to C7, C9 to C8, C10 to C9, DA1 to DA2, Q2 to Q1, Q4 to Q2, Q1 to Q4, Q3 to Q5, R2 to R1, R3 to R2, R1 to R3, R7 to R5, R5 to R6, R6 to R7
Connections:
- net labels added: ADC_LUM, MEAS_LUM
- wire segments 199 -> 208
- no-connect marks 25 -> 23
Other:
- moved on the sheet: ANT1, BLN1, C17, C19, C21, C24, C26, DD1, DD2, F1, L2, R1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

Commit message: HW2 sent to production
Connections:
- net BTN2: now also DD1.29 (MCO/CK1/PA8), SW4.1; no longer DD1.11 (ADC1/T2C2/PA1), SW3.1
- net BTN3: now also DD1.11 (ADC1/T2C2/PA1), SW3.1; no longer DD1.29 (MCO/CK1/PA8), SW4.1
Changed lines of the file:
@@
 BTN1
 Text Label 6050 1500 2    60   ~ 0
-BTN2
+BTN3
 Text Label 5850 1600 0    60   ~ 0
 ADC_BATTERY
@@
 $EndComp
 Text Label 6050 2200 2    60   ~ 0
-BTN3
+BTN2
 Text Label 2650 2900 0    60   ~ 0
 WS_CTRL
@@
 BTN1
 Text Label 6200 7650 0    60   ~ 0
+BTN3
+Text Label 6200 8050 0    60   ~ 0
 BTN2
-Text Label 6200 8050 0    60   ~ 0
-BTN3
 $Comp
 L BUTTON SW2

Commit message: + Antenna matched
Parts:
- C24: value * -> 5.1pF
- C26: value * -> DoNotMount
- L2: value * -> 15nH
Changed lines of the file:
@@
 P 12950 2000
 F 0 "L2" V 12850 1860 40  0000 C CNN
-F 1 "*" V 12850 2000 40  0000 C CNN
+F 1 "15nH" V 12850 2000 40  0000 C CNN
 F 2 "Inductors:IND_0402" V 13010 2010 40  0001 C CNN
 F 3 "" V 12850 1860 60  0001 C CNN
@@
 P 12600 2500
 F 0 "C24" H 12500 2400 50  0000 L CNN
-F 1 "*" H 12500 2600 50  0000 L CNN
+F 1 "5.1pF" H 12500 2600 50  0000 L CNN
 F 2 "Capacitors:CAP_0402" V 12700 2350 28  0001 C BNN
 F 3 "" H 12500 2400 60  0001 C CNN
@@
 P 13300 2500
 F 0 "C26" H 13200 2400 50  0000 L CNN
-F 1 "*" H 13200 2600 50  0000 L CNN
+F 1 "DoNotMount" H 13200 2600 50  0000 L CNN
 F 2 "Capacitors:CAP_0402" V 13400 2350 28  0001 C BNN
 F 3 "" H 13200 2400 60  0001 C CNN

Commit message: + IFA antenna
Parts:
- removed ANT1: ANT_PCB_MONO, Radio:ANT_868_ARMLETG, symbol ANT_PCB_MONO
- removed DA1: NCP583SQ, SOT:SC82AB, symbol NCP583SQ
- removed DD1: STM32L151CxTx, LQFP_TQFP:LQFP48, symbol STM32L151CxTx
- removed HOLE4, HOLE6: HOLE_METALLED, PCB:Hole2d4_out4d5mm, symbol HOLE_METALLED
- removed R7: 10k, Resistors:RES_0603, symbol R
- added ANT1: AntIFAMushroom, Radio:ANT_IFA_MUSHROOM, symbol ANT_GENERAL
- added C29: 1u, Capacitors:CAP_0603, symbol C
- added DA1: MCP1700, SOT:SOT23-3, symbol MCP1700
- added DD1: STM32F030C8Tx, LQFP_TQFP:LQFP48, symbol STM32F030C8Tx
- added XL14, XL15: CONN_3, Connectors:PLS-3, symbol CONN_3
- C14, C2: value 220pF -> 0.1u
- C23: value 0.1u -> 10u
- C24: value 5.1pF -> *
- C26: value DoNotMount -> 100pF
- C4, C9: value 10n -> 0.1u
- C5: value 0.1u -> *; footprint Capacitors:CAP_0603 -> Capacitors:CAP_0402; Price (none) -> 0.5; SolderPoints (none) -> 2
- C6: value 3.3pF -> 0.1u
- L2: value 15nH -> *
- Q2: value IRLML9303 -> IRLML6401
- R5: value 20k -> 56k
- R8: value 10k -> 100k
- SW1: value SWITCH -> SS-9; footprint BtnsSwitches:SW_SS-1P2T -> BtnsSwitches:SW_SS9
Connections:
- net +3.3V: now also DA1.2 (OUT), DD1.1 (VDD), DD1.24 (VDD), DD1.48 (VDD), DD1.9 (VDDA), XL14.2 (PM), XL15.2 (PM); no longer C5.1
- net +BATT: now also DA1.3 (IN)
- net ADC_BATTERY: now also DD1.12 (ADC2/T15C1/TX2/PA2)
- net ADC_LUM: now also DD1.18 (PB0/T3C3/T1C2N/ADC8)
- net ANT1: now also C26.1; no longer BLN1.1 (Unbal)
- net ANT2: now also C5.1, ANT1.1 (RF); no longer C26.1
- net BTN1: now also DD1.10 (ADC0/WKUP1/PA0)
- net BTN2: now also DD1.29 (MCO/CK1/T1C1/PA8)
- net BTN3: now also DD1.11 (ADC1/PA1)
- net CC_CS: now also DD1.14 (ADC4/T14C1/CK2/PA4)
- net CC_GDO0: now also DD1.13 (ADC3/T15C2/RX2/PA3)
- net CC_MISO: now also DD1.16 (ADC6/T16C1/T3C1/MISO1/PA6)
- net CC_MOSI: now also DD1.17 (ADC7/T14C1/T17C1/T1C1N/T3C2/MOSI1/PA7)
- net CC_SCK: now also DD1.15 (ADC5/SCK1/PA5)
- net GND: now also DA2.1 (~OE), ANT1.2 (GND), C29.2, DA1.1 (GND), DD1.23 (VSS), DD1.44 (BOOT0), DD1.47 (VSS), DD1.8 (VSSA), XL14.1 (P1), XL15.1 (P1); no longer C26.2
- net MEAS_LUM: now also DD1.19 (PB1/T3C4/T14C1/T1C3N/ADC9)
- net NO_RADIO: now also DD1.43 (PB7/SDA1/T17C1N/RX1)
- net PWR_EN: now also DD1.27 (PB14/MISO2/T1C2N/T15C1)
- net SWCLK: now also DD1.37 (TX2/SWCLK/PA14)
- net SWDIO: now also DD1.34 (IROUT/SWDIO/PA13)
- net UART_RX: now also DD1.31 (T1C3/RX1/PA10)
- net UART_TX: now also DD1.30 (T1C2/TX1/PA9)
- net VCC: now also C29.1
- net WS_CTRL: now also DD1.28 (PB15/MOSI2/T1C3N/T15C1N/T15C2)
- net at TP1.1: now also DD1.7 (NRST)
- new net: BLN1.1 (Unbal), C26.2
- new net AUX1: DD1.40 (PB4/T3C1/MISO1), XL14.3
- new net AUX2: DD1.41 (PB5/T3C2/MOSI1), XL15.3
Other:
- note added: "Pins 24, 48, 1+9"
- note removed: "Pins 24, 36, 48, 1+9"
- moved on the sheet: BLN1, C15, C16, C17, C19, C21, C24, DD2, HOLE5, L2, R5, R6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

Commit message: + PCB v4
Parts:
- removed C5: *, Capacitors:CAP_0402, symbol C
- C24: value * -> 3pF
- L2: value * -> 3.3nH
Changed lines of the file:
@@
-$EndComp
-$Comp
-L CONN_1 XL2
-U 1 1 589A6890
-P 1200 9900
-F 0 "XL2" H 1278 9938 40  0000 L CNN
-F 1 "CONN_1" H 1278 9862 40  0000 L CNN
-F 2 "Connectors:PLS-1Rnd" H 1200 9900 60  0001 C CNN
-F 3 "" H 1200 9900 60  0000 C CNN
-	1    1200 9900
-	-1   0    0    -1
 $EndComp
 $Comp
 L GND #PWR021
 U 1 1 589A6BDD
-P 1550 10050
-F 0 "#PWR021" H 1640 10030 30  0001 C CNN
-F 1 "GND" H 1550 9970 30  0001 C CNN
-F 2 "" H 1550 10050 60  0001 C CNN
-F 3 "" H 1550 10050 60  0001 C CNN
-	1    1550 10050
+P 1550 10450
+F 0 "#PWR021" H 1640 10430 30  0001 C CNN
+F 1 "GND" H 1550 10370 30  0001 C CNN
+F 2 "" H 1550 10450 60  0001 C CNN
+F 3 "" H 1550 10450 60  0001 C CNN
+	1    1550 10450
 	1    0    0    -1
 $EndComp
@@
 P 13900 2050
 F 0 "L2" V 13800 1910 40  0000 C CNN
-F 1 "*" V 13800 2050 40  0000 C CNN
+F 1 "3.3nH" V 13800 2050 40  0000 C CNN
 F 2 "Inductors:IND_0402" V 13960 2060 40  0001 C CNN
 F 3 "" V 13800 1910 60  0001 C CNN
@@
 P 13550 2550
 F 0 "C24" H 13450 2450 50  0000 L CNN
-F 1 "*" H 13450 2650 50  0000 L CNN
+F 1 "3pF" H 13450 2650 50  0000 L CNN
 F 2 "Capacitors:CAP_0402" V 13650 2400 28  0001 C BNN
 F 3 "" H 13450 2450 60  0001 C CNN
@@
 	1450 9450 2200 9450
 Wire Wire Line
-	1550 9650 1550 10050
+	1550 9650 1550 10450
 Wire Wire Line
 	1450 9650 1550 9650
@@
 NoConn ~ 6100 3400
 $Comp
-L GND #PWR056
-U 1 1 5A09708E
-P 14200 2800
-F 0 "#PWR056" H 14290 2780 30  0001 C CNN
-F 1 "GND" H 14200 2720 30  0001 C CNN
-F 2 "" H 14200 2800 60  0001 C CNN
-F 3 "" H 14200 2800 60  0001 C CNN
-	1    14200 2800
-	1    0    0    -1
-$EndComp
-$Comp
-L C C5
-U 1 1 5A097096
-P 14200 2550
-F 0 "C5" H 14100 2450 50  0000 L CNN
-F 1 "*" H 14100 2650 50  0000 L CNN
-F 2 "Capacitors:CAP_0402" V 14300 2400 28  0001 C BNN
-F 3 "" H 14100 2450 60  0001 C CNN
-F 4 "0.5" H 14200 2550 60  0001 C CNN "Price"
-F 5 "2" H 14300 2650 60  0001 C CNN "SolderPoints"
-	1    14200 2550
-	1    0    0    -1
-$EndComp
-Wire Wire Line
-	14200 2750 14200 2800
-Wire Wire Line
-	14200 2050 14200 2350
-Connection ~ 14200 2050
-$Comp
 L ANT_GENERAL ANT1
 U 1 1 5A097C5D
@@
 	2350 5750 2350 5650
 Connection ~ 2350 5650
+$Comp
+L CONN_1 XL2
+U 1 1 589A6890
+P 1200 9900
+F 0 "XL2" H 1278 9938 40  0000 L CNN
+F 1 "CONN_1" H 1278 9862 40  0000 L CNN
+F 2 "Connectors:PLS-1Rnd" H 1200 9900 60  0001 C CNN
+F 3 "" H 1200 9900 60  0000 C CNN
+	1    1200 9900
+	-1   0    0    -1
+$EndComp
 $EndSCHEMATC

Commit message: Smth
Parts:
- ANT1: symbol ANT_GENERAL -> Antennas_kl:ANT_GENERAL
- BLN1: symbol BALUN868JOHANSON -> RFICs:BALUN868JOHANSON
- C1, C10, C11, C12, C13, C14, C15, C16, C17, C18, C19, C2, C20, C21, C22, C23, C24, C25, C26, C27, C28, C29, C3, C4, C6, C7, C8, C9: symbol C -> Tittar_kl:C
- DA1: symbol MCP1700 -> Power_kl:MCP1700
- DA2: symbol MC74VHC1 -> standard_logic:MC74VHC1
- DD1: symbol STM32F030C8Tx -> st_kl:STM32F030C8Tx
- DD2: symbol CC1101 -> RFICs:CC1101
- F1: symbol Fuse0R -> Tittar_kl:Fuse0R
- HOLE1, HOLE2, HOLE3, HOLE5: symbol HOLE_METALLED -> pcb_details:HOLE_METALLED
- L1, L2: symbol L -> Tittar_kl:L
- Logo1: symbol Logo -> pcb_details:Logo
- Q1: symbol N_3PIN -> Transistors_kl:N_3PIN
- Q2: symbol P_3PIN -> Transistors_kl:P_3PIN
- Q3: symbol Phototransistor -> Transistors_kl:Phototransistor
- Q4, Q5, Q6: symbol LED_RGB_WS2812B -> Tittar_kl:LED_RGB_WS2812B
- R1, R2, R3, R4, R5, R6, R8: symbol R -> Tittar_kl:R
- RP1, RP2, RP3, RP4: symbol REFPOINT -> pcb_details:REFPOINT
- SW1: symbol SWITCH -> mushroom-rescue:SWITCH-RESCUE-mushroom
- SW2, SW3, SW4: symbol BUTTON -> mushroom-rescue:BUTTON-RESCUE-mushroom
- TP1, TP2: symbol TESTPOINT -> pcb_details:TESTPOINT
- XL1: symbol CONN_6 -> Connectors_kl:CONN_6
- XL10, XL12, XL14, XL15, XL4, XL6, XL8: symbol CONN_3 -> Connectors_kl:CONN_3
- XL11, XL13, XL2, XL5, XL7, XL9: symbol CONN_1 -> Connectors_kl:CONN_1
- XL3: symbol CONN_2 -> Connectors_kl:CONN_2
- XTAL1: symbol CRYSTAL_H -> Tittar_kl:CRYSTAL_H
Connections:
- wire segments 210 -> 267
