File: Mushroom_hw/mushroom.sch (KiCad schematic (older format))
At the start: 81 parts, among them Q1 2N7002, Q2 IRLML6401, Q3 ALS-PT19-315C, Q4 LED_RGB_WS2812B, Q5 LED_RGB_WS2812B, Q6 LED_RGB_WS2812B, SW1 SS-9, SW2 BUTTON, SW3 BUTTON, SW4 BUTTON

Commit message: + HW v5
Parts:
- removed C27, C28: 0.1u, Capacitors:CAP_0603, symbol Tittar_kl:C
- removed DA2: MC74VHC1, SOT:SOT23-5, symbol standard_logic:MC74VHC1
- removed DD1: STM32F030C8Tx, LQFP_TQFP:LQFP48, symbol st_kl:STM32F030C8Tx
- removed F1: Fuse0R, Resistors:RES_0603_FUSE, symbol Tittar_kl:Fuse0R
- removed Q1: 2N7002, SOT:SOT23-3, symbol Transistors_kl:N_3PIN
- removed Q2: IRLML6401, SOT:SOT23-3, symbol Transistors_kl:P_3PIN
- removed Q4, Q5, Q6: LED_RGB_WS2812B, LEDs:LED_WS2812B, symbol Tittar_kl:LED_RGB_WS2812B
- removed RP3, RP4: REFPOINT, PCB:REF_POINT_1MM, symbol pcb_details:REFPOINT
- removed XL10, XL12, XL4, XL6, XL8: CONN_3, Connectors:PLS-3, symbol Connectors_kl:CONN_3
- removed XL11, XL13, XL5, XL7, XL9: CONN_1, Connectors:SIL1_ROUND_1MM8, symbol Connectors_kl:CONN_1
- added C5: 0.1u, Capacitors:CAP_0603, symbol Tittar_kl:C
- added D1: PMEG2020, Diodes:SOD323, symbol Tittar_kl:D_Shottky
- added DA2, DA3: ULN200x, SO_DIL_TSSOP:SO16_150MIL, symbol Transistors_kl:ULN200x
- added DD1: STM32L151CxTx, LQFP_TQFP:LQFP48, symbol st_kl:STM32L151CxTx
- added HOLE4, HOLE6, HOLE7, HOLE8: HOLE_METALLED, PCB:Hole2d2_out3d5mm, symbol pcb_details:HOLE_METALLED
- added Q1, Q2, Q4: LED_5050_new, LEDs:LED_5050, symbol Tittar_kl:LED_5050_new
- added R10, R11, R12, R13, R14, R16, R17, R18, R7, R9: 100R, Resistors:RES_0603, symbol Tittar_kl:R
- added R15: 56k, Resistors:RES_0603, symbol Tittar_kl:R
- added R19: 1k, Resistors:RES_0603, symbol Tittar_kl:R
- added R20: 1M, Resistors:RES_0603, symbol Tittar_kl:R
- added R21: 2R0, Resistors:RES_0603, symbol Tittar_kl:R
- added XL10, XL4, XL6, XL8: CONN_4, Connectors:WB-04(MW-4M), symbol Connectors_kl:CONN_4
- added XL5: USB_MICRO_2H, Connectors:USBmicro_MOLEX_1050170001, symbol Connectors_kl:USB_MINI_B
- added XTAL2: 12MHz, Quartz:03225C4, symbol Tittar_kl:CRYSTAL_H
- ANT1: footprint Radio:ANT_IFA_MUSHROOM -> Antennas:ANT_IFA_MUSHROOM
- C18, C20: value 10u -> 18pF; PN CL10A106MQ8NNNC -> (none); Price 2.5 -> 0.5; URL https://www.terraelectronica.ru/catalog.php?ID=1155&search=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 -> (none)
- C22: value 0.1u -> 10n; Price (none) -> 0.5; SolderPoints (none) -> 2
- C25: value 0.1u -> 2u2; Price (none) -> 0.5; SolderPoints (none) -> 2
- DA1: footprint SOT:SOT23-3 -> SOT:SOT23-3A
- HOLE1, HOLE2, HOLE3, HOLE5: footprint PCB:Hole2d4_out4d5mm -> PCB:Hole2d2_out3d5mm
- Q3: footprint Resistors:RES_0603 -> Resistors:RES_0805
- R3, R4: value 100k -> 100R
- RP1, RP2: footprint PCB:REF_POINT_1MM -> PCB:REF_POINT_2MM
- SW1: symbol mushroom-rescue:SWITCH-RESCUE-mushroom -> Switches:SWITCH_H
- SW2, SW3, SW4: symbol mushroom-rescue:BUTTON-RESCUE-mushroom -> Switches:BUTTON
Connections:
- net labels added: B1, B2, B3, B4, BO1, BO2, BO3, BO4, D+, D-, G1, G2, G3, G4, GO1, GO2, GO3, GO4, MEASURE_EN, R1, R2, R3, R4, RO1, RO2, RO3, RO4
- net labels removed: DIN0, DIN1, DIN2, DIN3, DIN4, MEAS_LUM, NO_RADIO, PWR_EN, PwrUnst, WS_CTRL
- wire segments 267 -> 345
- no-connect marks 23 -> 8
Other:
- note added: "Pins 24, 36, 48, 1+9"
- note added: "T2C1"
- note added: "T2C2"
- note added: "T3C1"
- note added: "T3C2"
- note added: "T3C3"
- note added: "T3C4"
- note added: "T4C1"
- note added: "T4C2"
- note added: "T4C3"
- note added: "T4C4"
- note added: "T9C1"
- note added: "T9C2"
- note removed: "Extra transistor is required \nto eliminate fantom powering of MCU"
- note removed: "Pins 24, 48, 1+9"
- note removed: "Power switch"
- note removed: "Solder when radio not mounted\nto disable power-on check"
- note removed: "WS2812 control"
- moved on the sheet: C1, C10, C11, C12, C13, C14, C15, C16, C2, C23, C29, C3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

Commit message: Sch fixed
Parts:
- BLN1: symbol RFICs:BALUN868JOHANSON -> RF_ICs:BALUN868JOHANSON
- DD2: symbol RFICs:CC1101 -> RF_ICs:CC1101
Connections:
- net BAT_IN: now also D1.C
- net at R21.2, XL5.1 (UVcc): now also D1.A
- net +3.3V renamed +3v3
Other:
- moved on the sheet: L1, L2
Changed lines of the file:
@@
 EESchema Schematic File Version 4
 LIBS:mushroom-cache
-EELAYER 26 0
+EELAYER 29 0
 EELAYER END
 $Descr A3 16535 11693
@@
 $EndComp
 $Comp
-L power:+3.3V #PWR06
-U 1 1 53285E86
-P 5350 9450
-F 0 "#PWR06" H 5350 9410 30  0001 C CNN
-F 1 "+3.3V" H 5430 9480 30  0000 C CNN
-F 2 "" H 5350 9450 60  0001 C CNN
-F 3 "" H 5350 9450 60  0001 C CNN
-	1    5350 9450
-	1    0    0    -1
-$EndComp
-$Comp
 L power:PWR_FLAG #FLG07
 U 1 1 53285E9F
@@
 U 1 1 589C2FA9
 P 4850 7550
-F 0 "L1" V 4700 7400 40  0000 C CNN
+F 0 "L1" V 4950 7400 40  0000 C CNN
 F 1 "BLM15AG102SN1" V 4750 7550 40  0000 C CNN
 F 2 "Inductors:IND_0402" V 4910 7560 40  0001 C CNN
 F 3 "" H 4850 7550 60  0000 C CNN
 	1    4850 7550
-	0    1    1    0
+	0    1    -1   0
 $EndComp
 $Comp
@@
 $EndComp
 $Comp
-L RFICs:CC1101 DD2
+L RF_ICs:CC1101 DD2
 U 1 1 589C304B
 P 10600 2700
@@
 U 1 1 589C3078
 P 13900 2050
-F 0 "L2" V 13800 1910 40  0000 C CNN
-F 1 "3.3nH" V 13800 2050 40  0000 C CNN
+F 0 "L2" V 14000 1900 40  0000 C CNN
+F 1 "3.3nH" V 14000 2100 40  0000 C CNN
 F 2 "Inductors:IND_0402" V 13960 2060 40  0001 C CNN
 F 3 "" V 13800 1910 60  0001 C CNN
@@
 F 5 "2" V 14000 2110 60  0001 C CNN "SolderPoints"
 	1    13900 2050
-	0    1    1    0
+	0    1    -1   0
 $EndComp
 $Comp
@@
 $EndComp
 $Comp
-L RFICs:BALUN868JOHANSON BLN1
+L RF_ICs:BALUN868JOHANSON BLN1
 U 1 1 589C30EA
 P 12000 2150
@@
 $EndComp
 NoConn ~ 9850 2650
-$Comp
-L power:+3.3V #PWR058
-U 1 1 589C3147
-P 900 7550
-F 0 "#PWR058" H 900 7510 30  0001 C CNN
-F 1 "+3.3V" H 980 7580 30  0000 C CNN
-F 2 "" H 900 7550 60  0001 C CNN
-F 3 "" H 900 7550 60  0001 C CNN
-	1    900  7550
-	-1   0    0    -1
-$EndComp
 Text Label 6550 1400 2    60   ~ 0
 BTN1
@@
 $EndComp
 $Comp
-L power:+3.3V #PWR067
-U 1 1 589E25DA
-P 9600 9100
-F 0 "#PWR067" H 9600 9060 30  0001 C CNN
-F 1 "+3.3V" H 9680 9130 30  0000 C CNN
-F 2 "" H 9600 9100 60  0001 C CNN
-F 3 "" H 9600 9100 60  0001 C CNN
-	1    9600 9100
-	1    0    0    -1
-$EndComp
-$Comp
-L power:+3.3V #PWR068
-U 1 1 589E4315
-P 4500 7550
-F 0 "#PWR068" H 4500 7510 30  0001 C CNN
-F 1 "+3.3V" H 4580 7580 30  0000 C CNN
-F 2 "" H 4500 7550 60  0001 C CNN
-F 3 "" H 4500 7550 60  0001 C CNN
-	1    4500 7550
-	-1   0    0    -1
-$EndComp
-$Comp
-L power:+3.3V #PWR069
-U 1 1 589E5028
-P 3300 3750
-F 0 "#PWR069" H 3300 3710 30  0001 C CNN
-F 1 "+3.3V" H 3380 3780 30  0000 C CNN
-F 2 "" H 3300 3750 60  0001 C CNN
-F 3 "" H 3300 3750 60  0001 C CNN
-	1    3300 3750
-	-1   0    0    -1
-$EndComp
-$Comp
 L Switches:BUTTON SW3
 U 1 1 589E6745
@@
 $EndComp
 $Comp
-L power:+3.3V #PWR070
-U 1 1 589E674B
-P 9650 10500
-F 0 "#PWR070" H 9650 10460 30  0001 C CNN
-F 1 "+3.3V" H 9730 10530 30  0000 C CNN
-F 2 "" H 9650 10500 60  0001 C CNN
-F 3 "" H 9650 10500 60  0001 C CNN
-	1    9650 10500
-	1    0    0    -1
-$EndComp
-$Comp
 L Switches:BUTTON SW4
 U 1 1 589E680D
@@
 	1    0    0    -1
 $EndComp
-$Comp
-L power:+3.3V #PWR071
-U 1 1 589E6813
-P 9650 10900
-F 0 "#PWR071" H 9650 10860 30  0001 C CNN
-F 1 "+3.3V" H 9730 10930 30  0000 C CNN
-F 2 "" H 9650 10900 60  0001 C CNN
-F 3 "" H 9650 10900 60  0001 C CNN
-	1    9650 10900
-	1    0    0    -1
-$EndComp
 Text Notes 8950 8700 0    60   ~ 0
 Buttons
@@
 $EndComp
 $Comp
-L power:+3.3V #PWR076
+L power:+3v3 #PWR076
 U 1 1 58A0EC2C
 P 1450 1000
 F 0 "#PWR076" H 1450 960 30  0001 C CNN
-F 1 "+3.3V" H 1530 1030 30  0000 C CNN
+F 1 "+3v3" H 1530 1030 30  0000 C CNN
 F 2 "" H 1450 1000 60  0001 C CNN
 F 3 "" H 1450 1000 60  0001 C CNN
@@
 $EndComp
 $Comp
-L power:+3.3V #PWR078
-U 1 1 589B07CB
-P 9350 7450
-F 0 "#PWR078" H 9350 7410 30  0001 C CNN
-F 1 "+3.3V" H 9430 7480 30  0000 C CNN
-F 2 "" H 9350 7450 60  0001 C CNN
-F 3 "" H 9350 7450 60  0001 C CNN
-	1    9350 7450
-	-1   0    0    1
-$EndComp
-$Comp
 L Transistors_kl:Phototransistor Q3
 U 1 1 589B07D1
@@
 Wire Wire Line
 	1000 2400 1000 2250
-$Comp
-L power:+3.3V #PWR025
-U 1 1 5A0772BB
-P 1100 2150
-F 0 "#PWR025" H 1100 2110 30  0001 C CNN
-F 1 "+3.3V" H 1180 2180 30  0000 C CNN
-F 2 "" H 1100 2150 60  0001 C CNN
-F 3 "" H 1100 2150 60  0001 C CNN
-	1    1100 2150
-	1    0    0    -1
-$EndComp
 Wire Wire Line
 	1100 2150 1000 2150
@@
 Wire Wire Line
 	1000 3100 1000 2950
-$Comp
-L power:+3.3V #PWR028
-U 1 1 5A07823B
-P 1100 2850
-F 0 "#PWR028" H 1100 2810 30  0001 C CNN
-F 1 "+3.3V" H 1180 2880 30  0000 C CNN
-F 2 "" H 1100 2850 60  0001 C CNN
-F 3 "" H 1100 2850 60  0001 C CNN
-	1    1100 2850
-	1    0    0    -1
-$EndComp
 Wire Wire Line
 	1100 2850 1000 2850
@@
 	1    0    0    -1
 $EndComp
-Wire Wire Line
-	6900 9700 7000 9700
 Connection ~ 6900 9700
-Wire Wire Line
-	7400 9700 7500 9700
 $Comp
 L power:GND #PWR059
@@
 Wire Wire Line
 	6500 10400 6500 10500
-Wire Bus Line
-	9200 1600 9200 2550
 Connection ~ 6500 10500
 Wire Wire Line
 	6500 10500 6600 10500
+$Comp
+L power:+3v3 #PWR?
+U 1 1 5CEB5F3F
+P 1100 2850
+F 0 "#PWR?" H 1100 2810 30  0001 C CNN
+F 1 "+3v3" H 1180 2880 30  0000 C CNN
+F 2 "" H 1100 2850 60  0001 C CNN
+F 3 "" H 1100 2850 60  0001 C CNN
+	1    1100 2850
+	1    0    0    -1
+$EndComp
+$Comp
+L power:+3v3 #PWR?
+U 1 1 5CED8E02
+P 1100 2150
+F 0 "#PWR?" H 1100 2110 30  0001 C CNN
+F 1 "+3v3" H 1180 2180 30  0000 C CNN
+F 2 "" H 1100 2150 60  0001 C CNN
+F 3 "" H 1100 2150 60  0001 C CNN
+	1    1100 2150
+	1    0    0    -1
+$EndComp
+$Comp
+L power:+3v3 #PWR?
+U 1 1 5CF1DDF0
+P 3300 3750
+F 0 "#PWR?" H 3300 3710 30  0001 C CNN
+F 1 "+3v3" H 3380 3780 30  0000 C CNN
+F 2 "" H 3300 3750 60  0001 C CNN
+F 3 "" H 3300 3750 60  0001 C CNN
+	1    3300 3750
+	-1   0    0    -1
+$EndComp
+$Comp
+L power:+3v3 #PWR?
+U 1 1 5CF84E09
+P 4500 7550
+F 0 "#PWR?" H 4500 7510 30  0001 C CNN
+F 1 "+3v3" H 4580 7580 30  0000 C CNN
+F 2 "" H 4500 7550 60  0001 C CNN
+F 3 "" H 4500 7550 60  0001 C CNN
+	1    4500 7550
+	-1   0    0    -1
+$EndComp
+$Comp
+L power:+3v3 #PWR?
+U 1 1 5CFA7EE5
+P 900 7550
+F 0 "#PWR?" H 900 7510 30  0001 C CNN
+F 1 "+3v3" H 980 7580 30  0000 C CNN
+F 2 "" H 900 7550 60  0001 C CNN
+F 3 "" H 900 7550 60  0001 C CNN
+	1    900  7550
+	-1   0    0    -1
+$EndComp
+$Comp
+L power:+3v3 #PWR?
+U 1 1 5D031FFA
+P 5350 9450
+F 0 "#PWR?" H 5350 9410 30  0001 C CNN
+F 1 "+3v3" H 5430 9480 30  0000 C CNN
+F 2 "" H 5350 9450 60  0001 C CNN
+F 3 "" H 5350 9450 60  0001 C CNN
+	1    5350 9450
+	1    0    0    -1
+$EndComp
+Wire Wire Line
+	6900 9700 7050 9700
+Wire Wire Line
+	7350 9700 7500 9700
+$Comp
+L power:+3v3 #PWR?
+U 1 1 5D0BCEDB
+P 9650 10500
+F 0 "#PWR?" H 9650 10460 30  0001 C CNN
+F 1 "+3v3" H 9730 10530 30  0000 C CNN
+F 2 "" H 9650 10500 60  0001 C CNN
+F 3 "" H 9650 10500 60  0001 C CNN
+	1    9650 10500
+	1    0    0    -1
+$EndComp
+$Comp
+L power:+3v3 #PWR?
+U 1 1 5D0DFCCA
+P 9600 9100
+F 0 "#PWR?" H 9600 9060 30  0001 C CNN
+F 1 "+3v3" H 9680 9130 30  0000 C CNN
+F 2 "" H 9600 9100 60  0001 C CNN
+F 3 "" H 9600 9100 60  0001 C CNN
+	1    9600 9100
+	1    0    0    -1
+$EndComp
+$Comp
+L power:+3v3 #PWR?
+U 1 1 5D1029B1
+P 9650 10900
+F 0 "#PWR?" H 9650 10860 30  0001 C CNN
+F 1 "+3v3" H 9730 10930 30  0000 C CNN
+F 2 "" H 9650 10900 60  0001 C CNN
+F 3 "" H 9650 10900 60  0001 C CNN
+	1    9650 10900
+	1    0    0    -1
+$EndComp
+$Comp
+L power:+3v3 #PWR?
+U 1 1 5D18B2DA
+P 9350 7450
+F 0 "#PWR?" H 9350 7410 30  0001 C CNN
+F 1 "+3v3" H 9430 7480 30  0000 C CNN
+F 2 "" H 9350 7450 60  0001 C CNN
+F 3 "" H 9350 7450 60  0001 C CNN
+	1    9350 7450
+	-1   0    0    -1
+$EndComp
+Wire Bus Line
+	9200 1600 9200 2550
 $EndSCHEMATC
