File: Mushroom_hw/mushroom.kicad_pcb (KiCad board)
At the start: 2 copper layers, 48 x 85 mm, 82 parts, among them Q1 2N7002, Q2 IRLML6401, Q3 ALS-PT19-315C, Q4 LED_RGB_WS2812B, Q5 LED_RGB_WS2812B, Q6 LED_RGB_WS2812B, SW1 SS-9, SW2 BUTTON, SW3 BUTTON, SW4 BUTTON

Commit message: + HW v5
Parts:
- removed C27, C28: 0.1u, Capacitors:CAP_0603
- removed F1: Fuse0R, Resistors:RES_0603_FUSE
- removed Q5, Q6: LED_RGB_WS2812B, LEDs:LED_WS2812B
- removed RP3, RP4: REFPOINT, PCB:REF_POINT_1MM
- removed XL11, XL13, XL7, XL9: CONN_1, Connectors:SIL1_ROUND_1MM8
- removed XL12: CONN_3, Connectors:PLS-3
- added D1: PMEG2020, Diodes:SOD323, F.Cu at (220.6, 179.0)
- added DA3: ULN200x, SO_DIL_TSSOP:SO16_150MIL, F.Cu at (227.3, 170.8)
- added HOLE4: HOLE_METALLED, PCB:Hole2d2_out3d5mm, F.Cu at (228.0, 143.0)
- added HOLE6: HOLE_METALLED, PCB:Hole2d2_out3d5mm, F.Cu at (237.0, 155.0)
- added HOLE7: HOLE_METALLED, PCB:Hole2d2_out3d5mm, F.Cu at (219.0, 155.0)
- added HOLE8: HOLE_METALLED, PCB:Hole2d2_out3d5mm, F.Cu at (228.0, 159.5)
- added R10: 100R, Resistors:RES_0603, F.Cu at (248.8, 173.3)
- added R11: 100R, Resistors:RES_0603, F.Cu at (248.8, 174.9)
- added R12: 100R, Resistors:RES_0603, F.Cu at (234.0, 166.9)
- added R13: 100R, Resistors:RES_0603, F.Cu at (234.0, 168.5)
- added R14: 100R, Resistors:RES_0603, F.Cu at (234.0, 170.1)
- added R15: 56k, Resistors:RES_0603, F.Cu at (218.8, 165.8)
- added R16: 100R, Resistors:RES_0603, F.Cu at (234.0, 171.7)
- added R17: 100R, Resistors:RES_0603, F.Cu at (234.0, 173.3)
- added R18: 100R, Resistors:RES_0603, F.Cu at (234.0, 174.9)
- added R19: 1k, Resistors:RES_0603, F.Cu at (218.8, 169.0)
- added R20: 1M, Resistors:RES_0603, F.Cu at (220.6, 180.6)
- added R21: 2R0, Resistors:RES_0603, F.Cu at (235.4, 180.6)
- added R7: 100R, Resistors:RES_0603, F.Cu at (248.8, 170.1)
- added R9: 100R, Resistors:RES_0603, F.Cu at (248.8, 171.7)
- added XTAL2: 12MHz, Quartz:03225C4, F.Cu at (218.4, 171.8)
- ANT1: footprint Radio:ANT_IFA_MUSHROOM -> Antennas:ANT_IFA_MUSHROOM
- C18, C20: value 10u -> 18pF
- C22: value 0.1u -> 10n
- C24: value * -> 3pF
- C25: value 0.1u -> 2u2
- C5: value * -> 0.1u; footprint Capacitors:CAP_0402 -> Capacitors:CAP_0603
- DA1: footprint SOT:SOT23-3 -> SOT:SOT23-3A
- DA2: value MC74VHC1 -> ULN200x; footprint SOT:SOT23-5 -> SO_DIL_TSSOP:SO16_150MIL
- DD1: value STM32F030C8Tx -> STM32L151CxTx
- HOLE1, HOLE2, HOLE3, HOLE5: footprint PCB:Hole2d4_out4d5mm -> PCB:Hole2d2_out3d5mm
- L2: value * -> 3.3nH
- Q1: value 2N7002 -> LED_5050_new; footprint SOT:SOT23-3 -> LEDs:LED_5050
- Q2: value IRLML6401 -> LED_5050_new; footprint SOT:SOT23-3 -> LEDs:LED_5050
- Q3: footprint Resistors:RES_0603 -> Resistors:RES_0805
- Q4: value LED_RGB_WS2812B -> LED_5050_new; footprint LEDs:LED_WS2812B -> LEDs:LED_5050
- R3, R4: value 100k -> 100R
- RP1, RP2: footprint PCB:REF_POINT_1MM -> PCB:REF_POINT_2MM
- XL10, XL4, XL6, XL8: value CONN_3 -> CONN_4; footprint Connectors:PLS-3 -> Connectors:WB-04(MW-4M); moved to B.Cu
- XL5: value CONN_1 -> USB_MICRO_2H; footprint Connectors:SIL1_ROUND_1MM8 -> Connectors:USBmicro_MOLEX_1050170001; moved to B.Cu
- moved HOLE3 87.2 mm to (254.0, 120.5)
- moved Q3 72.1 mm to (256.8, 133.7), turned to 90 degrees
- moved R8 69.0 mm to (254.0, 133.5), turned to 270 degrees
- moved C23 66.4 mm to (252.0, 133.5), turned to 270 degrees
- moved XL10 54.1 mm to (200.5, 132.5), turned to 90 degrees
- moved XL8 51.2 mm to (194.5, 132.5), turned to 90 degrees
- moved C10 44.6 mm to (201.6, 150.9)
- moved C7 44.6 mm to (203.5, 150.9)
- moved DA1 44.6 mm to (206.3, 150.9)
- moved C16 43.8 mm to (206.3, 156.2), turned to 180 degrees
- moved C15 43.7 mm to (206.3, 154.5), turned to 180 degrees
- moved HOLE1 43.1 mm to (202.0, 120.5)
- moved SW2 41.3 mm to (258.0, 148.5)
- moved SW1 38.5 mm to (196.0, 162.5), turned to 270 degrees
- moved XL3 38.4 mm to (199.5, 176.0), turned to 315 degrees
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Connections:
- C18 pad 1: GND -> Net-(C18-Pad1)
- C18 pad 2: PwrUnst -> GND
- C20 pad 1: GND -> Net-(C20-Pad1)
- C20 pad 2: PwrUnst -> GND
- C22 pad 1: PwrUnst -> Net-(C22-Pad1)
- C25 pad 1: PwrUnst -> GND
- C25 pad 2: GND -> Net-(C25-Pad2)
- C5 pad 1: /ANT2 -> +3.3V
- DA2 pad 1: GND -> /R1
- DA2 pad 2: /WS_CTRL -> /G1
- DA2 pad 3: GND -> /B1
- DA2 pad 4: /DIN0 -> /R2
- DA2 pad 5: PwrUnst -> /G2
- DD1 pad 11: /BTN3 -> /R1
- DD1 pad 12: /ADC_BATTERY -> /G1
- DD1 pad 13: /CC_GDO0 -> /B1
- DD1 pad 14: /CC_CS -> /ADC_BATTERY
- DD1 pad 15: /CC_SCK -> /R2
- DD1 pad 16: /CC_MISO -> /G2
- DD1 pad 17: /CC_MOSI -> /B2
- DD1 pad 18: /ADC_LUM -> /R3
- DD1 pad 19: /MEAS_LUM -> /G3
- DD1 pad 2: Net-(DD1-Pad2) -> (no net)
- DD1 pad 20: Net-(DD1-Pad20) -> /CC_GDO0
- DD1 pad 21: Net-(DD1-Pad21) -> /AUX1
- DD1 pad 22: Net-(DD1-Pad22) -> /AUX2
- DD1 pad 25: Net-(DD1-Pad25) -> /ADC_LUM
- DD1 pad 26: Net-(DD1-Pad26) -> /CC_SCK
- DD1 pad 27: /PWR_EN -> /CC_MISO
- DD1 pad 28: /WS_CTRL -> /CC_MOSI
- DD1 pad 29: /BTN2 -> /MEASURE_EN
- DD1 pad 3: Net-(DD1-Pad3) -> /BTN2
- DD1 pad 32: Net-(DD1-Pad32) -> /D-
- DD1 pad 33: Net-(DD1-Pad33) -> /D+
- DD1 pad 35: Net-(DD1-Pad35) -> GND
- DD1 pad 36: Net-(DD1-Pad36) -> +3.3V
- DD1 pad 38: Net-(DD1-Pad38) -> (no net)
- DD1 pad 39: Net-(DD1-Pad39) -> (no net)
- DD1 pad 4: Net-(DD1-Pad4) -> /BTN3
- DD1 pad 40: /AUX1 -> (no net)
- DD1 pad 41: /AUX2 -> /CC_CS
- DD1 pad 42: Net-(DD1-Pad42) -> /B3
- DD1 pad 43: /NO_RADIO -> /R4
- DD1 pad 45: Net-(DD1-Pad45) -> /G4
- DD1 pad 46: Net-(DD1-Pad46) -> /B4
- DD1 pad 5: Net-(DD1-Pad5) -> Net-(C20-Pad1)
- DD2 pad 3: Net-(DD2-Pad3) -> (no net)
- Q1 pad 1: /PWR_EN -> /BO1
- Q1 pad 2: GND -> /GO1
- Q1 pad 3: Net-(Q1-Pad3) -> /RO1
- Q2 pad 1: Net-(Q1-Pad3) -> /BO2
- Q2 pad 2: +BATT -> /GO2
- Q2 pad 3: PwrUnst -> /RO2
- Q4 pad 1: PwrUnst -> /BO3
- Q4 pad 2: Net-(Q4-Pad2) -> /GO3
- Q4 pad 3: GND -> /RO3
- Q4 pad 4: /DIN0 -> +BATT
- R1 pad 1: PwrUnst -> +BATT
- R2 pad 2: GND -> Net-(DA2-Pad10)
- R3 pad 1: /PWR_EN -> Net-(DA2-Pad16)
- R3 pad 2: GND -> /RO1
- R4 pad 1: +BATT -> Net-(DA2-Pad15)
- R4 pad 2: Net-(Q1-Pad3) -> /GO1
- R8 pad 2: /MEAS_LUM -> /MEASURE_EN
- SW1 pad 3: Net-(SW1-Pad3) -> (no net)
- SW1 pad H: (no net) -> GND
- XL10 pad 1: /DIN3 -> +BATT
- XL10 pad 2: PwrUnst -> /RO4
- XL10 pad 3: /DIN4 -> /GO4
- XL4 pad 1: /DIN0 -> +BATT
- XL4 pad 2: PwrUnst -> /RO1
- XL4 pad 3: /DIN1 -> /GO1
- XL5 pad 1: GND -> Net-(D1-PadA)
- XL6 pad 1: /DIN1 -> +BATT
- XL6 pad 2: PwrUnst -> /RO2
- XL6 pad 3: /DIN2 -> /GO2
- XL8 pad 1: /DIN2 -> +BATT
- XL8 pad 2: PwrUnst -> /RO3
- XL8 pad 3: /DIN3 -> /GO3
Routing:
- net +BATT: track 18.7 -> 135.9 mm, vias 0 -> 7
- net PwrUnst: track 116.2 -> 0.00 mm, vias 2 -> 0
- net /MEASURE_EN: track 0.00 -> 78.1 mm, vias 0 -> 4
- net /BO1: track 0.00 -> 73.5 mm, vias 0 -> 2
- net /GO1: track 0.00 -> 71.8 mm, vias 0 -> 2
- net /BO2: track 0.00 -> 70.5 mm, vias 0 -> 3
- net /GO2: track 0.00 -> 70.1 mm, vias 0 -> 2
- net /RO1: track 0.00 -> 69.9 mm, vias 0 -> 2
- net /BO3: track 0.00 -> 66.7 mm, vias 0 -> 2
- net /RO2: track 0.00 -> 64.0 mm, vias 0 -> 2
- net /BO4: track 0.00 -> 63.3 mm, vias 0 -> 2
- net /GO3: track 0.00 -> 63.0 mm, vias 0 -> 2
- net /GO4: track 0.00 -> 59.8 mm, vias 0 -> 2
- net /RO3: track 0.00 -> 59.3 mm, vias 0 -> 2
- net /RO4: track 0.00 -> 55.6 mm, vias 0 -> 2
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Other:
- board size 48 x 85 mm -> 72 x 72 mm
- net class Default: trace_width 0.25 -> 0.22
- board text added: "+3V3"
- board text added: "+3v3"
- board text added: "Crystal Mushroom v5"
- board text added: "ON"
- board text added: "USB"
- board text removed: "3V3 Power Supply"
- board text removed: "Crystal Mushroom v4"
- board text removed: "In"
- board text removed: "LED Power Control"
- board text removed: "LED5"
- board text removed: "Level Shifter"
- board text removed: "MCU"
- board text removed: "Out"
- board text removed: "Solder if radio not mounted"

Commit message: + Sch + PCB Sent to factory
Parts:
- removed C29: 1u, Capacitors:CAP_0603
- removed DA3: ULN200x, SO_DIL_TSSOP:SO16_150MIL
- removed HOLE6, HOLE7, HOLE8: HOLE_METALLED, PCB:Hole2d2_out3d5mm
- removed Q2: LED_5050_new, LEDs:LED_5050
- removed Q3: ALS-PT19-315C, Resistors:RES_0805
- removed SW4: BUTTON, BtnsSwitches:BTN_6x6_4x4
- removed TP1: TESTPOINT, PCB:TESTPOINT_1MM
- removed XL10: CONN_4, Connectors:WB-04(MW-4M)
- removed XL14, XL15: CONN_3, Connectors:PLS-3
- added C27: *, Capacitors:CAP_0402, B.Cu at (152.0, 112.0)
- added L3: *, Inductors:IND_0402, B.Cu at (150.8, 110.7)
- added R22: 1k, Resistors:RES_0603, B.Cu at (133.6, 105.1)
- added R23: 1k, Resistors:RES_0603, B.Cu at (109.5, 99.5)
- added R24: 1k, Resistors:RES_0603, B.Cu at (118.9, 99.5)
- added R25: 1k, Resistors:RES_0603, B.Cu at (120.5, 99.5)
- added R26: 1k, Resistors:RES_0603, B.Cu at (123.7, 98.8)
- added R27: 56k, Resistors:RES_0603, B.Cu at (137.2, 108.9)
- added TP4: TESTPOINT, PCB:TESTPOINT_1MM, B.Cu at (140.8, 110.4)
- added XL7: CONN_4, Connectors:WB-04(MW-4M), B.Cu at (131.0, 101.2)
- added XL9: CONN_4, Connectors:WB-04(MW-4M), B.Cu at (123.4, 95.6)
- ANT1: value AntIFAMushroom -> ANT_PCB_MONO; footprint Antennas:ANT_IFA_MUSHROOM -> Antennas:Firefly_868; moved to B.Cu
- BLN1, D1, DD2, L1, R19, TP2: moved to B.Cu
- C1: value 10u -> 2u2; footprint Capacitors:CAP_0603 -> Capacitors:CAP_0603_Silks; moved to B.Cu
- C10: value 10u -> 1u; footprint Capacitors:CAP_0603 -> Capacitors:CAP_0603_Silks; moved to B.Cu
- C11: value 10n -> 0.1u; footprint Capacitors:CAP_0603 -> Capacitors:CAP_0603_Silks; moved to B.Cu
- C12, C3, C4, C5, C6: footprint Capacitors:CAP_0603 -> Capacitors:CAP_0603_Silks; moved to B.Cu
- C13: value 1u -> 0.1u; footprint Capacitors:CAP_0603 -> Capacitors:CAP_0603_Silks; moved to B.Cu
- C14, C2, C9: value 0.1u -> 10u; footprint Capacitors:CAP_0603 -> Capacitors:CAP_0603_Silks; moved to B.Cu
- C15: value 0.1u -> 18pF; footprint Capacitors:CAP_0603 -> Capacitors:CAP_0603_Silks; moved to B.Cu
- C16, C23: value 10u -> 18pF; footprint Capacitors:CAP_0603 -> Capacitors:CAP_0603_Silks; moved to B.Cu
- C17, C18, C19: value 18pF -> 0.1u; footprint Capacitors:CAP_0603 -> Capacitors:CAP_0603_Silks; moved to B.Cu
- C20: value 18pF -> 1u; footprint Capacitors:CAP_0603 -> Capacitors:CAP_0603_Silks; moved to B.Cu
- C21, C7: value 0.1u -> 1u; footprint Capacitors:CAP_0603 -> Capacitors:CAP_0603_Silks; moved to B.Cu
- C22: value 10n -> 18pF; footprint Capacitors:CAP_0603 -> Capacitors:CAP_0603_Silks; moved to B.Cu
- C24: value 3pF -> 0.1u; footprint Capacitors:CAP_0402 -> Capacitors:CAP_0603_Silks; moved to B.Cu
- C25: value 2u2 -> 0.1u; footprint Capacitors:CAP_0603 -> Capacitors:CAP_0603_Silks; moved to B.Cu
- C26: value 100pF -> *; moved to B.Cu
- C8: value 0.1u -> 10n; footprint Capacitors:CAP_0603 -> Capacitors:CAP_0603_Silks; moved to B.Cu
- DA1: value MCP1700 -> TP4056; footprint SOT:SOT23-3A -> SO_DIL_TSSOP:SO8_150MIL; moved to B.Cu
- DA2: value ULN200x -> MCP1700; footprint SO_DIL_TSSOP:SO16_150MIL -> SOT:SOT23-3A; moved to B.Cu
- DD1: value STM32L151CxTx -> STM32F072RxTx; footprint LQFP_TQFP:LQFP48 -> LQFP_TQFP:LQFP64; moved to B.Cu
- HOLE1, HOLE2, HOLE3, HOLE4, HOLE5: footprint PCB:Hole2d2_out3d5mm -> PCB:Hole2d4_out4d4mm
- L2: value 3.3nH -> BLM15AG102SN1; moved to B.Cu
- Logo1: footprint Pictures:Ostranna_12d7_10d1 -> Pictures:Ostranna_16d9_13d5; moved to B.Cu
- Q1: value LED_5050_new -> IRLML6401; footprint LEDs:LED_5050 -> SOT:SOT23-3; moved to B.Cu
- Q4: value LED_5050_new -> 2N7002; footprint LEDs:LED_5050 -> SOT:SOT23-3; moved to B.Cu
- R1: value 100k -> 10k; moved to B.Cu
- R10, R11, R12: value 100R -> 100k; moved to B.Cu
- R13, R14, R16, R18, R3, R7: value 100R -> 1k; moved to B.Cu
- R15, R5: value 56k -> 1k; moved to B.Cu
- R17: value 100R -> 2R0; moved to B.Cu
- R2: value 100k -> 0R2; footprint Resistors:RES_0603 -> Resistors:RES_1206; moved to B.Cu
- R20: value 1M -> 1k; moved to B.Cu
- R21: value 2R0 -> 1k; moved to B.Cu
- R4: value 100R -> 10k; moved to B.Cu
- R6: value 56k -> 1k2; moved to B.Cu
- R8: value 100k -> 1k; moved to B.Cu
- R9: value 100R -> 56k; moved to B.Cu
- RP1, RP2: footprint PCB:REF_POINT_2MM -> PCB:REF_POINT_1MM; moved to B.Cu
- SW1: value SS-9 -> BUTTON; footprint BtnsSwitches:SW_SS9 -> BtnsSwitches:BTN_4x4_SMD; moved to F.Cu
- SW2, SW3: footprint BtnsSwitches:BTN_6x6_4x4 -> BtnsSwitches:BTN_4x4_SMD
- XL1: value CONN_6 -> CONN_2; footprint Connectors:PLS-6 -> Connectors:SLD_2_2D5; moved to F.Cu
- XL2: value CONN_1 -> CONN_6; footprint Connectors:PLS-1Rnd -> Connectors:PLS-6_LOCK; moved to B.Cu
- XL3: value CONN_2 -> USB_MICRO; footprint Connectors:W02_Pitch_2d54 -> Connectors:USBmicro_MOLEX_1050170001; moved to F.Cu
- XL5: value USB_MICRO_2H -> CONN_1; footprint Connectors:USBmicro_MOLEX_1050170001 -> Connectors:PLS-1Square
- XTAL1: value 27MHz -> 12MHz; moved to B.Cu
- XTAL2: value 12MHz -> 27MHz; moved to B.Cu
- moved R10 172.0 mm to (92.7, 101.2), turned to -90 degrees
- moved R11 171.4 mm to (96.6, 96.1), turned to 90 degrees
- moved R2 165.5 mm to (102.1, 100.6), turned to 90 degrees
- moved XL5 165.3 mm to (89.5, 93.8)
- moved R1 164.7 mm to (104.4, 99.5), turned to 90 degrees
- moved R12 159.3 mm to (90.6, 97.7), turned to -90 degrees
- moved R3 157.7 mm to (105.1, 101.9), turned to 180 degrees
- moved SW2 156.7 mm to (105.8, 111.4), turned to -30 degrees
- moved R4 154.8 mm to (105.4, 110.2), turned to 90 degrees
- moved DA2 154.1 mm to (100.6, 110.2), turned to 90 degrees
- moved SW3 152.2 mm to (114.0, 115.0), turned to -18 degrees
- moved R21 151.1 mm to (107.9, 99.5), turned to 90 degrees
- moved HOLE4 149.7 mm to (86.2, 95.0)
- moved R8 146.9 mm to (111.1, 99.5), turned to 90 degrees
- moved Q4 146.3 mm to (90.1, 101.2), turned to 90 degrees
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Connections:
- ANT1 pad 1: /ANT2 -> Net-(ANT1-Pad1)
- C1 pad 1: GND -> Net-(C1-Pad1)
- C1 pad 2: +3.3V -> GND
- C10 pad 1: +BATT -> VCC
- C11 pad 1: +3.3V -> VCC
- C13 pad 1: +3.3V -> VCC
- C14 pad 1: VCC -> GND
- C14 pad 2: GND -> +BATT
- C15 pad 1: +3.3V -> Net-(C15-Pad1)
- C16 pad 1: +3.3V -> Net-(C16-Pad1)
- C17 pad 1: Net-(C17-Pad1) -> VCC
- C18 pad 1: Net-(C18-Pad1) -> VCC
- C19 pad 1: Net-(C19-Pad1) -> VCC
- C2 pad 1: VCC -> GND
- C2 pad 2: GND -> +3v3
- C20 pad 1: Net-(C20-Pad1) -> /PWR_UNST
- C21 pad 1: GND -> +3v3
- C21 pad 2: Net-(C21-Pad2) -> GND
- C23 pad 1: /ADC_LUM -> Net-(C23-Pad1)
- C24 pad 1: /ANT1 -> GND
- C24 pad 2: GND -> Net-(C24-Pad2)
- C25 pad 1: GND -> +3v3
- C25 pad 2: Net-(C25-Pad2) -> GND
- C26 pad 1: /ANT1 -> Net-(BLN1-Pad1)
- C26 pad 2: Net-(BLN1-Pad1) -> GND
- C3 pad 1: +3.3V -> +3v3
- C4 pad 1: VCC -> +3v3
- C5 pad 1: +3.3V -> +3v3
- C6 pad 1: VCC -> +3v3
- C7 pad 1: +BATT -> /MCU_VDDA
- C8 pad 1: +3.3V -> /MCU_VDDA
- C9 pad 1: VCC -> GND
- C9 pad 2: GND -> /5V_MID
- D1 pad A: Net-(D1-PadA) -> /5V_USB
- D1 pad C: /BAT_IN -> /PWR_UNST
- DA1 pad 2: +3.3V -> Net-(DA1-Pad2)
- DA1 pad 3: +BATT -> GND
- DA2 pad 1: /R1 -> GND
- DA2 pad 2: /G1 -> +3v3
- DA2 pad 3: /B1 -> /PWR_UNST
- DD1 pad 1: +3.3V -> +3v3
- DD1 pad 10: /BTN1 -> /ADC_BAT_EN
- DD1 pad 11: /R1 -> /IS_CHARGING
- DD1 pad 12: /G1 -> GND
- DD1 pad 13: /B1 -> /MCU_VDDA
- DD1 pad 14: /ADC_BATTERY -> /BTN_PWR
- DD1 pad 15: /R2 -> /R1
- DD1 pad 16: /G2 -> /G1
- DD1 pad 17: /B2 -> /B1
- DD1 pad 18: /R3 -> GND
- DD1 pad 19: /G3 -> +3v3
- DD1 pad 2: (no net) -> Net-(DD1-Pad2)
- DD1 pad 20: /CC_GDO0 -> /CC_CS
- DD1 pad 21: /AUX1 -> /CC_SCK
- DD1 pad 22: /AUX2 -> /CC_MISO
- DD1 pad 23: GND -> /CC_MOSI
- DD1 pad 24: +3.3V -> (no net)
- DD1 pad 25: /ADC_LUM -> (no net)
- DD1 pad 26: /CC_SCK -> /R2
- DD1 pad 27: /CC_MISO -> /G2
- DD1 pad 28: /CC_MOSI -> (no net)
- DD1 pad 29: /MEASURE_EN -> /B2
- DD1 pad 3: /BTN2 -> (no net)
- DD1 pad 30: /UART_TX -> /R3
- DD1 pad 31: /UART_RX -> GND
- DD1 pad 32: /D- -> +3v3
- DD1 pad 33: /D+ -> (no net)
- DD1 pad 34: /SWDIO -> (no net)
- DD1 pad 35: GND -> (no net)
- DD1 pad 36: +3.3V -> (no net)
- DD1 pad 37: /SWCLK -> /G3
- DD1 pad 38: (no net) -> /B3
- DD1 pad 4: /BTN3 -> Net-(DD1-Pad4)
- DD1 pad 41: /CC_CS -> /R4
- DD1 pad 42: /B3 -> /G4
- DD1 pad 43: /R4 -> /B4
- DD1 pad 44: GND -> /USB_DM
- DD1 pad 45: /G4 -> /USB_DP
- DD1 pad 46: /B4 -> /SWDIO
- DD1 pad 48: +3.3V -> +3v3
- DD1 pad 5: Net-(C20-Pad1) -> Net-(C15-Pad1)
- DD1 pad 7: Net-(DD1-Pad7) -> (no net)
- DD1 pad 8: GND -> /CC_GDO0
- DD1 pad 9: +3.3V -> /ADC_BAT
- DD2 pad 10: Net-(C19-Pad1) -> Net-(C23-Pad1)
- DD2 pad 5: Net-(C21-Pad2) -> Net-(C24-Pad2)
- DD2 pad 8: Net-(C17-Pad1) -> Net-(C22-Pad1)
- HOLE1 pad H: GND -> (no net)
- L1 pad 1: VCC -> +3v3
- L1 pad 2: +3.3V -> /MCU_VDDA
- L2 pad 1: /ANT2 -> VCC
- L2 pad 2: /ANT1 -> +3v3
- Q1 pad 1: /BO1 -> /5V_USB
- Q1 pad 2: /GO1 -> /PWR_UNST
- Q1 pad 3: /RO1 -> +BATT
- Q4 pad 1: /BO3 -> /ADC_BAT_EN
- Q4 pad 2: /GO3 -> GND
- Q4 pad 3: /RO3 -> Net-(Q4-Pad3)
- R1 pad 1: +BATT -> /5V_USB
- R1 pad 2: /ADC_BATTERY -> GND
- R10 pad 1: Net-(DA2-Pad12) -> /ADC_BAT_EN
- R10 pad 2: /GO2 -> GND
- R11 pad 1: Net-(DA2-Pad11) -> +BATT
- R11 pad 2: /BO2 -> /ADC_BAT
- R12 pad 1: Net-(DA3-Pad16) -> /ADC_BAT
- R12 pad 2: /RO3 -> Net-(Q4-Pad3)
- R13 pad 1: Net-(DA3-Pad15) -> /G1
- R13 pad 2: /GO3 -> Net-(R13-Pad2)
- R14 pad 1: Net-(DA3-Pad14) -> /G4
- R14 pad 2: /BO3 -> Net-(R14-Pad2)
- R15 pad 1: GND -> /B1
- R15 pad 2: /BTN1 -> Net-(R15-Pad2)
- R16 pad 1: Net-(DA3-Pad13) -> /B4
- R16 pad 2: /RO4 -> Net-(R16-Pad2)
- R17 pad 1: Net-(DA3-Pad12) -> /5V_USB
- R17 pad 2: /GO4 -> Net-(C1-Pad1)
- R18 pad 1: Net-(DA3-Pad11) -> /R2
- R18 pad 2: /BO4 -> Net-(R18-Pad2)
- R19 pad 1: Net-(C18-Pad1) -> /R5
- R19 pad 2: Net-(DD1-Pad6) -> Net-(R19-Pad2)
- R2 pad 1: /ADC_BATTERY -> /5V_USB
- R2 pad 2: Net-(DA2-Pad10) -> /5V_MID
- R20 pad 1: Net-(C22-Pad1) -> /G2
- R20 pad 2: GND -> Net-(R20-Pad2)
- R21 pad 1: Net-(C25-Pad2) -> /G5
- R21 pad 2: Net-(D1-PadA) -> Net-(R21-Pad2)
- R3 pad 1: Net-(DA2-Pad16) -> Net-(DD1-Pad2)
- R3 pad 2: /RO1 -> /5V_USB
- R4 pad 1: Net-(DA2-Pad15) -> /BTN_PWR
- R4 pad 2: /GO1 -> GND
- R5 pad 1: /CC_CS -> Net-(DD1-Pad6)
- R5 pad 2: VCC -> Net-(C16-Pad1)
- R6 pad 1: Net-(DD2-Pad17) -> Net-(DA1-Pad2)
- R7 pad 1: Net-(DA2-Pad14) -> /R1
- R7 pad 2: /BO1 -> Net-(R7-Pad2)
- R8 pad 1: /ADC_LUM -> /R4
- R8 pad 2: /MEASURE_EN -> Net-(R8-Pad2)
- R9 pad 1: Net-(DA2-Pad13) -> Net-(DD2-Pad17)
- R9 pad 2: /RO2 -> GND
- SW1 pad 1: +BATT -> /BTN_PWR
- SW1 pad 2: /BAT_IN -> +3v3
- SW2 pad 1: /BTN1 -> /BTN_L
- SW2 pad 2: +3.3V -> +3v3
- SW3 pad 1: /BTN3 -> /BTN_R
- SW3 pad 2: +3.3V -> +3v3
- TP2 pad 1: /CC_GDO0 -> Net-(DD1-Pad4)
- XL1 pad 1: +3.3V -> GND
- XL1 pad 2: /SWCLK -> +BATT
- XL2 pad 1: GND -> +3v3
- XL3 pad 1: /BAT_IN -> /5V_USB
- XL3 pad 2: GND -> /USB_DM
- XL4 pad 1: +BATT -> GND
- XL4 pad 2: /RO1 -> Net-(R15-Pad2)
- XL4 pad 3: /GO1 -> Net-(R13-Pad2)
- XL4 pad 4: /BO1 -> Net-(R7-Pad2)
- XL5 pad 1: Net-(D1-PadA) -> GND
- XL6 pad 1: +BATT -> GND
- XL6 pad 2: /RO2 -> Net-(R16-Pad2)
- XL6 pad 3: /GO2 -> Net-(R14-Pad2)
- XL6 pad 4: /BO2 -> Net-(R8-Pad2)
- XL8 pad 1: +BATT -> GND
- XL8 pad 2: /RO3 -> Net-(R23-Pad2)
- XL8 pad 3: /GO3 -> Net-(R21-Pad2)
- XL8 pad 4: /BO3 -> Net-(R19-Pad2)
- XTAL1 pad 1: Net-(C17-Pad1) -> Net-(C15-Pad1)
- XTAL1 pad 2: Net-(C19-Pad1) -> Net-(C16-Pad1)
- XTAL2 pad 1: Net-(C18-Pad1) -> Net-(C22-Pad1)
- XTAL2 pad 2: Net-(C20-Pad1) -> Net-(C23-Pad1)
Routing:
- net GND: track 969.9 -> 218.6 mm, vias 219 -> 105
- net +3.3V: track 193.4 -> 0.00 mm, vias 8 -> 0
- net +BATT: track 135.9 -> 15.3 mm, vias 7 -> 0
- net +3v3: track 0.00 -> 112.8 mm, vias 0 -> 8
- net /MEASURE_EN: track 78.1 -> 0.00 mm, vias 4 -> 0
- net /BO1: track 73.5 -> 0.00 mm, vias 2 -> 0
- net /GO1: track 71.8 -> 0.00 mm, vias 2 -> 0
- net /BO2: track 70.5 -> 0.00 mm, vias 3 -> 0
- net /GO2: track 70.1 -> 0.00 mm, vias 2 -> 0
- net /RO1: track 69.9 -> 0.00 mm, vias 2 -> 0
- net /BO3: track 66.7 -> 0.00 mm, vias 2 -> 0
- net /5V_USB: track 0.00 -> 66.1 mm, vias 0 -> 7
- net /RO2: track 64.0 -> 0.00 mm, vias 2 -> 0
- net /BO4: track 63.3 -> 0.00 mm, vias 2 -> 0
- net /GO3: track 63.0 -> 0.00 mm, vias 2 -> 0
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- added copper zone on B.Cu, net /5V_USB
- added copper zone on F.Cu, net /5V_USB
- added copper zone on In1.Cu, net GND
- added copper zone on In2.Cu, net GND
Other:
- board size 72 x 72 mm -> 94.7 x 33.9 mm
- copper layers 2 -> 4
- net class Default removed
- net class Wide removed
- rule pad_to_mask_clearance: 0.1 -> 0.06
- board text added: "Ostranna Mushroom v6"
- board text removed: "+3V3"
- board text removed: "+3v3"
- board text removed: "-"
- board text removed: "AUX1"
- board text removed: "AUX2"
- board text removed: "Btn1"
- board text removed: "Btn2"
- board text removed: "Btn3"
- board text removed: "Crystal Mushroom v5"
- board text removed: "E"
- board text removed: "LED A"
- board text removed: "LED B"
- board text removed: "LED C"
- board text removed: "LED2"
- board text removed: "LED3"
- board text removed: "LED4"
- board text removed: "Light detector"
- board text removed: "ON"
- board text removed: "Ostranna"
- board text removed: "Radio"
- board text removed: "USB"
